File: cvcart-dip/cvcart-dip.sch (KiCad schematic (older format))
At the start: 1 part

Commit message: working on schematic
Parts:
- added CON101: CV-EDGE, db-vgparts:CV-EDGE, symbol CV-EDGE
- added D101, D102: BAT54A, symbol BAT54A
- added U101: W27C512, db-dipics:DIP-28-600MIL, symbol W27C512
- gave numbers to parts that had none: 1
Connections:
- net labels added: +5V, A0, A1, A10, A11, A12, A13, A14, A2, A3, A4, A5, A6, A7, A8, A9, D0, D1, D2, D3, D4, D5, D6, D7, GND, ~8000, ~A000, ~C000, ~E000
- wire segments 0 -> 70
Other:
- moved on the sheet: R101

Commit message: netlist and pcb work
Parts:
- added C101: C, db-smt:0603, symbol C
- D101, D102: footprint (none) -> db-smt:SOT23
- R101: footprint (none) -> db-smt:0603
Connections:
- wire segments 70 -> 73
Changed lines of the file:
@@
 F 0 "R101" V 5900 5700 50  0000 C CNN
 F 1 "10k" V 5700 5675 50  0000 C CNN
-F 2 "" V 5730 5700 30  0000 C CNN
+F 2 "db-smt:0603" V 5730 5700 30  0001 C CNN
 F 3 "" H 5800 5700 30  0000 C CNN
 	1    5800 5700
@@
 $EndComp
 $Comp
-L +5V #PWR104
+L +5V #PWR01
 U 1 1 589B7390
 P 7700 4000
-F 0 "#PWR104" H 7700 3850 50  0001 C CNN
+F 0 "#PWR01" H 7700 3850 50  0001 C CNN
 F 1 "+5V" H 7700 4140 50  0000 C CNN
 F 2 "" H 7700 4000 50  0000 C CNN
@@
 $EndComp
 $Comp
-L GND #PWR105
+L GND #PWR02
 U 1 1 589B73AA
 P 7700 6250
-F 0 "#PWR105" H 7700 6000 50  0001 C CNN
+F 0 "#PWR02" H 7700 6000 50  0001 C CNN
 F 1 "GND" H 7700 6100 50  0000 C CNN
 F 2 "" H 7700 6250 50  0000 C CNN
@@
 $EndComp
 $Comp
-L +5V #PWR106
+L +5V #PWR03
 U 1 1 589B7417
-P 11150 5400
-F 0 "#PWR106" H 11150 5250 50  0001 C CNN
-F 1 "+5V" H 11150 5540 50  0000 C CNN
-F 2 "" H 11150 5400 50  0000 C CNN
-F 3 "" H 11150 5400 50  0000 C CNN
-	1    11150 5400
-	1    0    0    -1
-$EndComp
-$Comp
-L GND #PWR107
+P 11250 5350
+F 0 "#PWR03" H 11250 5200 50  0001 C CNN
+F 1 "+5V" H 11250 5490 50  0000 C CNN
+F 2 "" H 11250 5350 50  0000 C CNN
+F 3 "" H 11250 5350 50  0000 C CNN
+	1    11250 5350
+	1    0    0    -1
+$EndComp
+$Comp
+L GND #PWR04
 U 1 1 589B74AB
-P 11150 5700
-F 0 "#PWR107" H 11150 5450 50  0001 C CNN
-F 1 "GND" H 11150 5550 50  0000 C CNN
-F 2 "" H 11150 5700 50  0000 C CNN
-F 3 "" H 11150 5700 50  0000 C CNN
-	1    11150 5700
+P 11250 5950
+F 0 "#PWR04" H 11250 5700 50  0001 C CNN
+F 1 "GND" H 11250 5800 50  0000 C CNN
+F 2 "" H 11250 5950 50  0000 C CNN
+F 3 "" H 11250 5950 50  0000 C CNN
+	1    11250 5950
 	1    0    0    -1
 $EndComp
@@
 D0
 $Comp
-L GND #PWR103
+L GND #PWR05
 U 1 1 589B77FE
 P 6400 6250
-F 0 "#PWR103" H 6400 6000 50  0001 C CNN
+F 0 "#PWR05" H 6400 6000 50  0001 C CNN
 F 1 "GND" H 6400 6100 50  0000 C CNN
 F 2 "" H 6400 6250 50  0000 C CNN
@@
 $EndComp
 $Comp
-L GND #PWR102
+L GND #PWR06
 U 1 1 589B7887
 P 6050 4100
-F 0 "#PWR102" H 6050 3850 50  0001 C CNN
+F 0 "#PWR06" H 6050 3850 50  0001 C CNN
 F 1 "GND" H 6050 3950 50  0000 C CNN
 F 2 "" H 6050 4100 50  0000 C CNN
@@
 F 0 "D101" H 5025 5725 60  0000 C CNN
 F 1 "BAT54A" H 5075 5325 60  0000 C CNN
-F 2 "" H 5000 5600 60  0000 C CNN
+F 2 "db-smt:SOT23" H 5000 5600 60  0001 C CNN
 F 3 "" H 5000 5600 60  0000 C CNN
 	1    5000 5600
@@
 F 0 "D102" H 5025 6225 60  0000 C CNN
 F 1 "BAT54A" H 5075 5825 60  0000 C CNN
-F 2 "" H 5000 6100 60  0000 C CNN
+F 2 "db-smt:SOT23" H 5000 6100 60  0001 C CNN
 F 3 "" H 5000 6100 60  0000 C CNN
 	1    5000 6100
@@
 	7700 4100 7550 4100
 Wire Wire Line
-	10650 5400 11150 5400
-Wire Wire Line
-	10650 5500 11150 5500
-Wire Wire Line
-	11150 5500 11150 5700
+	10650 5400 11250 5400
 Wire Wire Line
 	5450 5675 5450 6175
@@
 ~8000
 $Comp
-L +5V #PWR101
+L +5V #PWR07
 U 1 1 589B87E6
 P 5800 5425
-F 0 "#PWR101" H 5800 5275 50  0001 C CNN
+F 0 "#PWR07" H 5800 5275 50  0001 C CNN
 F 1 "+5V" H 5800 5565 50  0000 C CNN
 F 2 "" H 5800 5425 50  0000 C CNN
@@
 Wire Wire Line
 	5800 5425 5800 5500
+$Comp
+L C C101
+U 1 1 589C79A7
+P 11250 5650
+F 0 "C101" H 11275 5750 50  0000 L CNN
+F 1 "C" H 11275 5550 50  0000 L CNN
+F 2 "db-smt:0603" H 11288 5500 30  0001 C CNN
+F 3 "" H 11250 5650 60  0000 C CNN
+	1    11250 5650
+	1    0    0    -1
+$EndComp
+Wire Wire Line
+	11250 5350 11250 5500
+Connection ~ 11250 5400
+Wire Wire Line
+	11250 5800 11250 5950
+Wire Wire Line
+	10650 5500 11025 5500
+Wire Wire Line
+	11025 5500 11025 5900
+Wire Wire Line
+	11025 5900 11250 5900
+Connection ~ 11250 5900
 $EndSCHEMATC
